File: The-GarlicBoard-2.1-ANSI.kicad_pcb (KiCad board)
At the start: 2 copper layers, 380 x 75.2 mm, 274 parts, among them J1 Molex Pico-EZMATE, J2 Molex Pico-EZMATE, J3 PAD_SQUARE_1MM, J4 PAD_SQUARE_1MM, J5 PAD_SQUARE_1MM, J6 PAD_SQUARE_1MM, J7 PAD_SQUARE_1MM, Q1 Q_PMOS_GSD, SW1 ESC, SW10 S, SW11 X, SW12 L_CMD, SW13 E, SW14 D, SW15 C, SW16 R, SW17 F, SW18 V, SW19 FN_1, SW2 TAB, SW20 T, SW21 G, SW22 B, SW23 Y, SW24 H, SW25 N, SW26 SPACE, SW27 U, SW28 J, SW29 M, SW3 L_SHIFT, SW30 I, SW31 K, SW32 COMMA, SW33 R_CMD, SW34 O, SW35 L, SW36 PERIOD, SW37 P, SW38 SEMI_COLON, SW39 SLASH, SW4 L_CTRL, SW40 R_ALT, SW41 HYPHEN, SW42 APOSTROPHE, SW43 R_SHIFT, SW44 R_CTRL, SW45 EQUALS, SW46 RETURN, SW47 FN_2, SW48 BCK_SPC, SW49 7, SW5 Q, SW50 4, SW51 1, SW52 00, SW53 8, SW54 5, SW55 2, SW56 0, SW57 9, SW58 6, SW59 3, SW6 A, SW60 NUM_PER, SW61 MINUS, SW62 PLUS, SW63 ENTER, SW64 PAD_LOCK, SW65 RotaryEncoder_Switch, SW66 SW_Push, SW67 SW_Push, SW7 Z, SW8 L_ALT, SW9 W, U1 RP2040, U3 W25Q128JVS, U5 NCP1117-3.3_SOT223, U6 AW20216SQNR, Y1 12MHz

Commit message: Final Pre-BOM changes
Parts:
- ST1, ST5: footprint marbastlib-mx:STAB_MX_P_3u -> marbastlib-mx:STAB_MX_3u
- ST2, ST3: footprint marbastlib-mx:STAB_MX_P_2.25u -> marbastlib-mx:STAB_MX_2.25u
- ST4: footprint marbastlib-mx:STAB_MX_P_2.75u -> marbastlib-mx:STAB_MX_2.75u
- moved J1 2.32 mm to (312.9, 128.5)
- renumbered BOOT to SW68
Routing:
- net DN: track 17.2 -> 24.5 mm
- net DP: track 17.3 -> 24.4 mm
- net Net-(J1-Pin_1): track 9.29 -> 11.6 mm
- net GND: vias 270 -> 276
Other:
- board text added: "TO OLED DISPLAY ONLY!"
- board text added: "TO UDB USB CONNECTOR ONLY!"
