File: The-GarlicBoard-2.1-ANSI.kicad_pcb (KiCad board)
At the start: 2 copper layers, 380 x 75.2 mm, 272 parts, among them J1 PAD_SQUARE_1MM, J2 Molex Pico-EZMATE, J3 PAD_SQUARE_1MM, J4 PAD_SQUARE_1MM, J5 PAD_SQUARE_1MM, J6 PAD_SQUARE_1MM, J7 Molex Pico-EZMATE, Q1 Q_PMOS_GSD, SW1 ESC, SW10 S, SW11 X, SW12 L_CMD, SW13 E, SW14 D, SW15 C, SW16 R, SW17 F, SW18 V, SW19 FN_1, SW2 TAB, SW20 T, SW21 G, SW22 B, SW23 Y, SW24 H, SW25 N, SW26 SPACE, SW27 U, SW28 J, SW29 M, SW3 L_SHIFT, SW30 I, SW31 K, SW32 COMMA, SW33 R_CMD, SW34 O, SW35 L, SW36 PERIOD, SW37 P, SW38 SEMI_COLON, SW39 SLASH, SW4 L_CTRL, SW40 R_ALT, SW41 HYPHEN, SW42 APOSTROPHE, SW43 R_CTRL, SW44 EQUALS, SW45 RETURN, SW46 FN_2, SW47 BCK_SPC, SW48 R_SHIFT, SW49 7, SW5 Q, SW50 4, SW51 1, SW52 00, SW53 8, SW54 5, SW55 2, SW56 0, SW57 9, SW58 6, SW59 3, SW6 A, SW60 NUM_PER, SW61 MINUS, SW62 PLUS, SW63 ENTER, SW64 PAD_LOCK, SW65 SW_Push, SW66 SW_Push, SW67 SW_Push, SW68 RotaryEncoder_Switch, SW7 Z, SW8 L_ALT, SW9 W, U1 RP2040, U2 W25Q128JVS, U3 NCP1117-3.3_SOT223, U4 AW20216SQNR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

Commit message: MAJOR REVISION
Completely remapped RGB LED matrix - previous version was completely wrong for the LEDs used!
Parts:
- RGB1, RGB10, RGB11, RGB12, RGB13, RGB14, RGB15, RGB16, RGB17, RGB18, RGB19, RGB2, RGB20, RGB21, RGB22, RGB23, RGB24, RGB25, RGB26, RGB27, RGB28, RGB29, RGB3, RGB30, RGB31, RGB32, RGB33, RGB34, RGB35, RGB36, RGB37, RGB38, RGB39, RGB4, RGB40, RGB41, RGB42, RGB43, RGB44, RGB45, RGB46, RGB47, RGB48, RGB49, RGB5, RGB50, RGB51, RGB52, RGB53, RGB54, RGB55, RGB56, RGB57, RGB58, RGB59, RGB6, RGB60, RGB61, RGB62, RGB63, RGB64, RGB7, RGB8, RGB9: footprint marbastlib-mx:LED_MX_6028R -> GarlicBoard v2:LED_MX_6028R FIXED
Routing:
- net Net-(RGB43-BK): track 365.4 -> 307.2 mm, vias 17 -> 14
- net Net-(RGB43-GK): track 342.0 -> 321.8 mm
- net Net-(RGB23-BK): track 297.6 -> 317.7 mm, vias 17 -> 15
- net Net-(RGB43-RK): track 341.0 -> 321.3 mm, vias 17 -> 16
- net Net-(RGB1-RK): track 477.2 -> 461.6 mm, vias 19 -> 17
- net Net-(RGB33-RK): track 256.1 -> 243.3 mm, vias 17 -> 18
- net COL7: track 167.0 -> 154.3 mm
- net COL8: track 205.4 -> 193.8 mm
- net COL5: track 222.2 -> 210.9 mm
- net Net-(RGB1-GK): track 472.0 -> 462.1 mm, vias 19 -> 17
- net COL0: track 466.3 -> 457.5 mm
- net Net-(RGB33-BK): track 256.5 -> 247.9 mm, vias 17 -> 18
- net Net-(RGB13-BK): track 358.9 -> 365.4 mm, vias 16 -> 15
- net Net-(RGB1-BK): track 469.8 -> 476.3 mm, vias 20 -> 16
- net SW7: track 371.1 -> 376.6 mm
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Other:
- board text added: "a different sort of keyboard by Thomas {dblquote}stiligFox{dblquote} Meyer (c) thomasmeyer 2025 v2.1_250713 ANSI"
- board text removed: "a different sort of keyboard by Thomas {dblquote}stiligFox{dblquote} Meyer (c) thomasmeyer 2025 v2.1_250705"
