File: The-GarlicBoard-2.1-ANSI.kicad_sch (KiCad schematic)
At the start: 273 parts, among them J1 Molex Pico-EZMATE, J2 Molex Pico-EZMATE, J3 PAD_SQUARE_1MM, J4 PAD_SQUARE_1MM, J5 PAD_SQUARE_1MM, J6 PAD_SQUARE_1MM, J7 PAD_SQUARE_1MM, Q1 Q_PMOS_GSD, SW1 ESC, SW10 S, SW11 X, SW12 L_CMD, SW13 E, SW14 D, SW15 C, SW16 R, SW17 F, SW18 V, SW19 FN_1, SW2 TAB, SW20 T, SW21 G, SW22 B, SW23 Y, SW24 H, SW25 N, SW26 SPACE, SW27 U, SW28 J, SW29 M, SW3 L_SHIFT, SW30 I, SW31 K, SW32 COMMA, SW33 R_CMD, SW34 O, SW35 L, SW36 PERIOD, SW37 P, SW38 SEMI_COLON, SW39 SLASH, SW4 L_CTRL, SW40 R_ALT, SW41 HYPHEN, SW42 APOSTROPHE, SW43 R_SHIFT, SW44 R_CTRL, SW45 EQUALS, SW46 RETURN, SW47 FN_2, SW48 BCK_SPC, SW49 7, SW5 Q, SW50 4, SW51 1, SW52 00, SW53 8, SW54 5, SW55 2, SW56 0, SW57 9, SW58 6, SW59 3, SW6 A, SW60 NUM_PER, SW61 MINUS, SW62 PLUS, SW63 ENTER, SW64 PAD_LOCK, SW65 RotaryEncoder_Switch, SW66 SW_Push, SW67 SW_Push, SW68 SW_Push, SW7 Z, SW8 L_ALT, SW9 W, U1 RP2040, U3 W25Q128JVS, U5 NCP1117-3.3_SOT223, U6 AW20216SQNR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

Commit message: Final Pre-BOM changes
Parts:
- ST1, ST5: footprint marbastlib-mx:STAB_MX_P_3u -> marbastlib-mx:STAB_MX_3u
- ST2, ST3: footprint marbastlib-mx:STAB_MX_P_2.25u -> marbastlib-mx:STAB_MX_2.25u
- ST4: footprint marbastlib-mx:STAB_MX_P_2.75u -> marbastlib-mx:STAB_MX_2.75u
Changed lines of the file:
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@@
 			)
 		)
-		(property "Footprint" "marbastlib-mx:STAB_MX_P_2.25u"
+		(property "Footprint" "marbastlib-mx:STAB_MX_2.25u"
 			(at 233.68 53.34 0)
 			(effects
@@
 			)
 		)
-		(property "Footprint" "marbastlib-mx:STAB_MX_P_3u"
+		(property "Footprint" "marbastlib-mx:STAB_MX_3u"
 			(at 233.68 68.58 0)
 			(effects
@@
 			)
 		)
-		(property "Footprint" "marbastlib-mx:STAB_MX_P_2.25u"
+		(property "Footprint" "marbastlib-mx:STAB_MX_2.25u"
 			(at 233.68 58.42 0)
 			(effects
@@
 			)
 		)
-		(property "Footprint" "marbastlib-mx:STAB_MX_P_3u"
+		(property "Footprint" "marbastlib-mx:STAB_MX_3u"
 			(at 233.68 48.26 0)
 			(effects
@@
 			)
 		)
-		(property "Footprint" "marbastlib-mx:STAB_MX_P_2.75u"
+		(property "Footprint" "marbastlib-mx:STAB_MX_2.75u"
 			(at 233.68 63.5 0)
 			(effects

Commit message: Parts update
Parts:
- C14: renamed from C23; LCSC C15525 -> C1713
- C16: renamed from C24; LCSC C15525 -> C1713
- C17: Basic or Extended (none) -> Basic; LCSC (none) -> C7171
- C18: renamed from C12; Basic or Extended (none) -> Basic; LCSC (none) -> C1592
- C19: renamed from C13; Basic or Extended (none) -> Basic; LCSC (none) -> C1525
- C20: renamed from C14; Basic or Extended (none) -> Basic; LCSC (none) -> C1525
- C21: renamed from C15; Basic or Extended (none) -> Basic; LCSC (none) -> C1592
- C22: renamed from C16; Basic or Extended (none) -> Basic; LCSC (none) -> C1525
- D1, D10, D11, D12, D13, D14, D15, D16, D17, D18, D19, D2, D20, D21, D22, D23, D24, D25, D26, D27, D28, D29, D3, D30, D31, D32, D33, D34, D35, D36, D37, D38, D39, D4, D40, D41, D42, D5, D6, D7, D8, D9: LCSC C191023 -> C282366
- D43: renamed from D44; LCSC C191023 -> C282366
- D44: renamed from D45; LCSC C191023 -> C282366
- D45: renamed from D46; LCSC C191023 -> C282366
- D46: renamed from D47; LCSC C191023 -> C282366
- D47: renamed from D48; LCSC C191023 -> C282366
- D48: renamed from D65; LCSC C191023 -> C282366
- D49: renamed from D43; LCSC C191023 -> C282366
- D50: renamed from D49; LCSC C191023 -> C282366
- D51: renamed from D50; LCSC C191023 -> C282366
- D52: renamed from D51; LCSC C191023 -> C282366
- D53: renamed from D52; LCSC C191023 -> C282366
- D54: renamed from D53; LCSC C191023 -> C282366
- D55: renamed from D54; LCSC C191023 -> C282366
- D56: renamed from D55; LCSC C191023 -> C282366
- D57: renamed from D56; LCSC C191023 -> C282366
- D58: renamed from D57; LCSC C191023 -> C282366
- D59: renamed from D58; LCSC C191023 -> C282366
- D60: renamed from D59; LCSC C191023 -> C282366
- D61: renamed from D60; LCSC C191023 -> C282366
- D62: renamed from D61; LCSC C191023 -> C282366
- D63: renamed from D62; LCSC C191023 -> C282366
- D64: renamed from D63; LCSC C191023 -> C282366
- D65: renamed from D64; LCSC C191023 -> C282366
- R10: renamed from R9; LCSC (none) -> C23140
- R11: renamed from R15; LCSC (none) -> C22973
- R12: renamed from R16; LCSC (none) -> C22973
- R13: renamed from R17; LCSC (none) -> C23140
- R14: renamed from R18; LCSC (none) -> C22973
- R15: renamed from R19; LCSC (none) -> C22973
- R16: renamed from R20; LCSC (none) -> C23140
- R17: renamed from R21; LCSC (none) -> C22973
- R18: renamed from R22; LCSC (none) -> C22973
- R19: renamed from R23; LCSC (none) -> C23140
- R20: renamed from R24; LCSC (none) -> C22973
- R21: renamed from R25; LCSC (none) -> C22973
- R22: renamed from R26; LCSC (none) -> C23140
- R23: renamed from R27; LCSC (none) -> C22973
- R24: renamed from R28; LCSC (none) -> C22973
- R28: renamed from R13; LCSC (none) -> C25531
- R7: renamed from R6; LCSC (none) -> C23140
- R8: renamed from R7; LCSC (none) -> C22973
- R9: renamed from R8; LCSC (none) -> C22973
- RGB1, RGB10, RGB11, RGB12, RGB13, RGB14, RGB15, RGB16, RGB17, RGB18, RGB19, RGB2, RGB20, RGB21, RGB22, RGB23, RGB24, RGB25, RGB26, RGB27, RGB28, RGB29, RGB3, RGB30, RGB31, RGB32, RGB33, RGB34, RGB35, RGB36, RGB37, RGB38, RGB39, RGB4, RGB40, RGB41, RGB42, RGB43, RGB44, RGB45, RGB46, RGB47, RGB48, RGB49, RGB5, RGB50, RGB51, RGB52, RGB53, RGB54, RGB55, RGB56, RGB57, RGB58, RGB59, RGB6, RGB60, RGB61, RGB62, RGB63, RGB64, RGB7, RGB8, RGB9: Basic or Extended (none) -> Extended; LCSC (none) -> C183826
- SW1, SW10, SW11, SW12, SW13, SW14, SW15, SW16, SW17, SW18, SW19, SW2, SW20, SW21, SW22, SW23, SW24, SW25, SW26, SW27, SW28, SW29, SW3, SW30, SW31, SW32, SW33, SW34, SW35, SW36, SW37, SW38, SW39, SW4, SW40, SW41, SW42, SW49, SW5, SW50, SW51, SW52, SW53, SW54, SW55, SW56, SW57, SW58, SW59, SW6, SW60, SW61, SW62, SW63, SW64, SW7, SW8, SW9: LCSC C5184526 -> C5156480
- SW43: renamed from SW44; LCSC C5184526 -> C5156480
- SW44: renamed from SW45; LCSC C5184526 -> C5156480
- SW45: renamed from SW46; LCSC C5184526 -> C5156480
- SW46: renamed from SW47; LCSC C5184526 -> C5156480
- SW47: renamed from SW48; LCSC C5184526 -> C5156480
- SW48: renamed from SW43; LCSC C5184526 -> C5156480
- SW65: renamed from SW68; LCSC C231329 -> C115351
- SW66: renamed from SW67; now left out of the parts list
- SW67: renamed from SW66; now left out of the parts list
- SW68: renamed from SW65; now left out of the parts list
- U4: renamed from U6; Basic or Extended (none) -> Extebded; LCSC (none) -> C7385556
- renumbered C20 to C12, C21 to C13, C22 to C15, H7 to H4, H4 to H5, H5 to H6, H6 to H7, J7 to J1, J1 to J7, R10 to R25, R11 to R26, R12 to R27, R14 to R6, U3 to U2, U5 to U3
Other:
- moved on the sheet: C1, C10, C11, C17, C18, C19, C2, C20, C21, C22, C3, C4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

Commit message: Final Update
Parts:
- removed R4, R5: 2k, Resistor_SMD:R_0402_1005Metric, symbol Device:R
- C19, C20, C22: value 0.1uF -> 100nF
Connections:
- net +5V: now also C17.1, Q1.2 (S); no longer C17.2, Q1.3 (D)
- net GND: now also C17.2; no longer C17.1
- net at J7.1 (Pin_1): now also Q1.3 (D); no longer Q1.2 (S)
Other:
- note added: "May 1, 2022 - July 12, 2025"
- note removed: "May 1, 2022 - Jan 4, 2023"
- moved on the sheet: C1, C10, C11, C12, C13, C14, C15, C16, C17, C18, C19, C2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

Commit message: MAJOR REVISION
Completely remapped RGB LED matrix - previous version was completely wrong for the LEDs used!
Parts:
- RGB1, RGB10, RGB11, RGB12, RGB13, RGB14, RGB15, RGB16, RGB17, RGB18, RGB19, RGB2, RGB20, RGB21, RGB22, RGB23, RGB24, RGB25, RGB26, RGB27, RGB28, RGB29, RGB3, RGB30, RGB31, RGB32, RGB33, RGB34, RGB35, RGB36, RGB37, RGB38, RGB39, RGB4, RGB40, RGB41, RGB42, RGB43, RGB44, RGB45, RGB46, RGB47, RGB48, RGB49, RGB5, RGB50, RGB51, RGB52, RGB53, RGB54, RGB55, RGB56, RGB57, RGB58, RGB59, RGB6, RGB60, RGB61, RGB62, RGB63, RGB64, RGB7, RGB8, RGB9: footprint marbastlib-mx:LED_MX_6028R -> GarlicBoard v2:LED_MX_6028R FIXED
Other:
- moved on the sheet: C17, R10, R11, R12, R13, R14, R15, R16, R17, R18, R19, R20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
